Commit message: wip -adding links

File: RoboSpecs.urdf (robot description, URDF)
Before this commit: robot None, 1 links, 0 joints
Links:
- removed link my_link

Commit message: wip -mapping it out

File: RoboSpecs.urdf (robot description, URDF)
Before this commit: robot my_robot, 0 links, 0 joints
Links:
- added link None
Joints:
- added joint None: type None

Commit message: wip -outline

File: RoboSpecs.urdf (robot description, URDF)
Before this commit: robot my_robot, 1 links, 1 joints
Links:
- removed link None
- added link ; visual cylinder length=0.0 radius=0.0
Joints:
- removed joint None
- added joint : type , parent parent_link, child child_link, origin xyz=0.0 0.0 0.0 rpy=0.0 0.0 0.0, axis 0.0 0.0 0.0

Commit message: wip -urdf names

File: RoboSpecs.urdf (robot description, URDF)
Before this commit: robot my_robot, 1 links, 1 joints
Links:
- removed link 
- added link base_link; visual box size=0.0 0.0 0.0
- added link base_motor; visual cylinder length=0.0 radius=0.0
- added link elbow_case; visual cylinder length=0.0 radius=0.0
- added link elbow_motor; visual cylinder length=0.0 radius=0.0
- added link forearm; visual cylinder length=0.0 radius=0.0
- added link gripper_case; visual box size=0.0 0.0 0.0
- added link hand; visual box size=0.0 0.0 0.0
- added link left_gripper; visual box size=0.0 0.0 0.0
- added link right_gripper; visual box size=0.0 0.0 0.0
- added link shoulder_case; visual cylinder length=0.0 radius=0.0
- added link shoulder_motor; visual cylinder length=0.0 radius=0.0
- added link upper_arm; visual cylinder length=0.0 radius=0.0
- added link wrist_case; visual cylinder length=0.0 radius=0.0
- added link wrist_motor; visual cylinder length=0.0 radius=0.0
Joints:
- added joint base_motor_joint: type revolute, parent base_link, child base_motor, origin xyz=0.0 0.0 0.0 rpy=0.0 0.0 0.0, axis 0.0 0.0 0.0
- added joint left_gripper_joint: type prismatic, parent gripper_case, child left_gripper, origin xyz=0.0 0.0 0.0 rpy=0.0 0.0 0.0, axis 0.0 0.0 0.0
- added joint right_gripper_joint: type prismatic, parent gripper_case, child right_gripper, origin xyz=0.0 0.0 0.0 rpy=0.0 0.0 0.0, axis 0.0 0.0 0.0
- joint : child child_link -> gripper_case; parent parent_link -> hand

Commit message: inital sizes and positions

File: RoboSpecs.urdf (robot description, URDF)
Before this commit: robot my_robot, 14 links, 4 joints
Links:
- link base_link: geometry visual box size=0.38 0.215 0.025
- link base_motor: geometry visual cylinder length=0.05 radius=0.05
- link elbow_case: geometry visual box size=0.078 0.054 0.035
- link elbow_motor: geometry visual cylinder length=0.07 radius=0.012
- link forearm: geometry visual cylinder length=0.12 radius=0.0065
- link gripper_case: geometry visual box size=0.02854 0.065 0.04
- link hand: geometry visual box size=0.03 0.052 0.02408
- link left_gripper: geometry visual box size=0.02844 0.006 0.01935
- link right_gripper: geometry visual box size=0.02844 0.006 0.01935
- link shoulder_case: geometry visual box size=0.066 0.06 0.034
- link shoulder_motor: geometry visual cylinder length=0.081 radius=0.02
- link upper_arm: geometry visual box size=0.0245 0.07753 0.146
- link wrist_case: geometry visual box size=0.06 0.04136 0.02639
- link wrist_motor: geometry visual cylinder length=0.052 radius=0.01204
Joints:
- removed joint 
- added joint arm_wrist_joint: type fixed, parent forearm, child wrist_case, origin xyz=-0.06 0.0 0.0 rpy=0.0 0.0 0.0
- added joint base_motor_shoulder_joint: type fixed, parent base_motor, child shoulder_case, origin xyz=0.1738 0.0 0.025 rpy=0.0 0.0 0.0
- added joint elbow_joint: type revolute, parent elbow_case, child elbow_motor, origin xyz=0.024 0.0 0.0 rpy=0.0 0.0 0.0, axis 0.0 1 0.0
- added joint forearm_elbow_joint: type fixed, parent elbow_motor, child forearm, origin xyz=0.06 0.0 0.0 rpy=0.0 0.0 0.0
- added joint gripper_hand_joint: type fixed, parent hand, child gripper_case, origin xyz=0.03 0.0 0.0 rpy=0.0 0.0 0.0
- added joint shoudler_arm_joint: type fixed, parent shoulder_motor, child upper_arm, origin xyz=0.1738 0.0 0.0 rpy=0.0 0.0 0.0
- added joint shoudler_joint: type revolute, parent shoulder_case, child shoulder_motor, origin xyz=0.1738 0.0 0.0 rpy=0.0 0.0 0.0, axis 0.0 1 0.0
- added joint upperarm_elbow_joint: type fixed, parent upper_arm, child elbow_case, origin xyz=0.024 0.0 0.0 rpy=0.0 0.0 0.0
- added joint wrist_hand_joint: type fixed, parent wrist_motor, child hand, origin xyz=0.0 0.0 0.0 rpy=0.0 0.0 0.0
- added joint wrist_joint: type revolute, parent wrist_case, child wrist_motor, origin xyz=0.0 -0.0115 0.0 rpy=0.0 0.0 0.0, axis 0.0 1 0.0
- joint base_motor_joint: axis 0.0 0.0 0.0 -> 0.0 0.0 1; origin xyz=0.0 0.0 0.0 rpy=0.0 0.0 0.0 -> xyz=-0.147 0.0 0.025 rpy=0.0 0.0 0.0
- joint left_gripper_joint: origin xyz=0.0 0.0 0.0 rpy=0.0 0.0 0.0 -> xyz=0.02854 0.0 0.0 rpy=0.0 0.0 0.0
- joint right_gripper_joint: origin xyz=0.0 0.0 0.0 rpy=0.0 0.0 0.0 -> xyz=0.02854 0.0 0.0 rpy=0.0 0.0 0.0

Commit message: initial rotation limits

File: RoboSpecs.urdf (robot description, URDF)
Before this commit: robot my_robot, 14 links, 13 joints
Joints:
- joint base_motor_joint: limit (none) -> lower=-2.0944 upper=1.0472 effort=0.470736 velocity=4.76
- joint elbow_joint: limit (none) -> lower=-1.0472 upper=1.5708 effort= velocity=
- joint left_gripper_joint: limit (none) -> lower=0.0 upper=0.0165 effort= velocity=
- joint right_gripper_joint: limit (none) -> lower=0.0 upper=0.0165 effort= velocity=
- joint shoudler_joint: limit (none) -> lower=-1.5708 upper=1.5708 effort= velocity=
- joint wrist_joint: limit (none) -> lower=-1.5708 upper=1.5708 effort= velocity=

Commit message: intial effort and velcotiies

File: RoboSpecs.urdf (robot description, URDF)
Before this commit: robot my_robot, 14 links, 13 joints
Joints:
- joint base_motor_joint: limit lower=-2.0944 upper=1.0472 effort=0.470736 velocity=4.76 -> lower=-2.0944 upper=1.0472 effort=0.47 velocity=4.75
- joint elbow_joint: limit lower=-1.0472 upper=1.5708 effort= velocity= -> lower=-1.0472 upper=1.5708 effort=1.07 velocity=4.53
- joint left_gripper_joint: limit lower=0.0 upper=0.0165 effort= velocity= -> lower=0.0 upper=0.0165 effort=0.755 velocity=4.97
- joint right_gripper_joint: limit lower=0.0 upper=0.0165 effort= velocity= -> lower=0.0 upper=0.0165 effort=0.755 velocity=4.97
- joint shoudler_joint: limit lower=-1.5708 upper=1.5708 effort= velocity= -> lower=-1.5708 upper=1.5708 effort=1.94 velocity=5.49
- joint wrist_joint: limit lower=-1.5708 upper=1.5708 effort= velocity= -> lower=-1.5708 upper=1.5708 effort=0.755 velocity=4.36
